File: kicad/GB-Sync.sch (KiCad schematic (older format))
At the start: 4 parts

Commit message: Refactored with real Link Port measurements
Parts:
- conn1, conn2, conn3, conn5: symbol GBC_link_edge_connector -> sync:GBC_link_edge_connector
Connections:
- wire segments 12 -> 18
Changed lines of the file:
@@
-EESchema Schematic File Version 2
-LIBS:power
-LIBS:device
-LIBS:transistors
-LIBS:conn
-LIBS:linear
-LIBS:regul
-LIBS:74xx
-LIBS:cmos4000
-LIBS:adc-dac
-LIBS:memory
-LIBS:xilinx
-LIBS:microcontrollers
-LIBS:dsp
-LIBS:microchip
-LIBS:analog_switches
-LIBS:motorola
-LIBS:texas
-LIBS:intel
-LIBS:audio
-LIBS:interface
-LIBS:digital-audio
-LIBS:philips
-LIBS:display
-LIBS:cypress
-LIBS:siliconi
-LIBS:opto
-LIBS:atmel
-LIBS:contrib
-LIBS:valves
-LIBS:sync
+EESchema Schematic File Version 4
 LIBS:GB-Sync-cache
-EELAYER 25 0
+EELAYER 26 0
 EELAYER END
 $Descr A4 11693 8268
 encoding utf-8
 Sheet 1 1
-Title ""
-Date ""
-Rev ""
+Title "Syncross"
+Date "2018-10-02"
+Rev "2"
 Comp ""
-Comment1 ""
-Comment2 ""
+Comment1 "Original layout by rebb"
+Comment2 "Refinements by Poldet"
 Comment3 ""
 Comment4 ""
 $EndDescr
 $Comp
-L GBC_link_edge_connector conn2
+L sync:GBC_link_edge_connector conn2
 U 1 1 584782F1
 P 5350 2150
@@
 $EndComp
 $Comp
-L GBC_link_edge_connector conn1
+L sync:GBC_link_edge_connector conn1
 U 1 1 584783EF
 P 6300 1750
@@
 $EndComp
 $Comp
-L GBC_link_edge_connector conn5
+L sync:GBC_link_edge_connector conn5
 U 1 1 5847847E
 P 7050 3650
@@
 $EndComp
 $Comp
-L GBC_link_edge_connector conn3
+L sync:GBC_link_edge_connector conn3
 U 1 1 584784C8
 P 7050 2350
@@
 	-1   0    0    1
 $EndComp
-Connection ~ 5350 2400
-Connection ~ 5350 2500
-Connection ~ 5350 2050
 Wire Wire Line
-	5950 1750 5950 3650
-Connection ~ 5950 2000
-Connection ~ 5950 2500
-Wire Wire Line
-	6500 1750 6500 3850
+	6500 1750 6500 1950
 Wire Wire Line
 	6500 2550 7050 2550
@@
 Connection ~ 6500 1950
 Wire Wire Line
-	6050 1750 6050 3400
+	6050 1750 6050 2100
 Wire Wire Line
 	6050 2400 5350 2400
@@
 Wire Wire Line
 	5950 3650 7050 3650
+Wire Wire Line
+	6500 2550 6500 3850
+Wire Wire Line
+	6500 1950 6500 2550
+Wire Wire Line
+	6050 2100 6050 2400
+Wire Wire Line
+	6050 2400 6050 3400
+Wire Wire Line
+	5950 2150 5950 2350
+Wire Wire Line
+	5950 1750 5950 2150
+Wire Wire Line
+	5950 2350 5950 3650
 $EndSCHEMATC
